File: ErgoDone.sch (KiCad schematic (older format))
At the start: 62 parts, among them J1 USB, J2 3.5mm, J3 JMP, J4 JMP, SW0:10 SW0:3, SW0:11 SW0:2, SW0:12 SW0:1, SW0:7 SW0:6, SW0:8 SW0:5, SW0:9 SW0:4, SW1:10 SW1:3, SW1:11 SW1:2, SW1:12 SW1:1, SW1:13 SW1:0, SW1:9 SW1:4, SW2:10 SW2:3, SW2:11 SW2:2, SW2:12 SW2:1, SW2:13 SW2:0, SW2:7 SW2:6, SW2:8 SW2:5, SW2:9 SW2:4, SW3:10 SW3:3, SW3:11 SW3:2, SW3:12 SW3:1, SW3:13 SW3:0, SW3:8 SW3:5, SW3:9 SW3:4, SW4:10 SW4:3, SW4:11 SW4:2, SW4:12 SW4:1, SW4:13 SW4:0, SW4:7 SW4:6, SW4:8 SW4:5, SW4:9 SW4:4, SW5:10 SW5:3, SW5:11 SW5:2, SW5:12 SW5:1, SW5:13 SW5:0, SW5:7 SW5:6, SW5:8 SW5:5, SW5:9 SW5:4, U1 ProMicro, U2 MCP23017

Commit message: update to v1.3
Parts:
- removed D1:7, D1:8: D, symbol DIODE
- added D1, D11, D13, D15, D17, D19, D21, D23, D25, D27, D29, D3, D31, D33, D35, D37, D39, D41, D43, D45, D47, D49, D5, D51, D53, D55, D57, D59, D61, D63, D65, D67, D69, D7, D71, D73, D75, D77, D79, D9: DIODE, ErgoDone:D_1206_L, symbol DIODE-RESCUE-ErgoDone
- added D10, D12, D14, D16, D18, D2, D20, D22, D24, D26, D28, D30, D32, D34, D36, D38, D4, D40, D42, D44, D46, D48, D50, D52, D54, D56, D58, D6, D60, D62, D64, D66, D68, D70, D72, D74, D76, D78, D8, D80: DIODE, ErgoDone:D_1206_R, symbol DIODE-RESCUE-ErgoDone
- added D81, D82: DIODE, ErgoDone:DIODE_SX, symbol DIODE
- C1: footprint Capacitors_ThroughHole:C_Rect_L7_W2_P5 -> ErgoDone:C_Disc_D6_P5
- J1: footprint (none) -> ErgoDone:USBMINImod
- J2: footprint (none) -> ErgoDone:4pin35mmAudio
- J3, J4: footprint (none) -> ErgoDone:100PITCH1X3
- LED_A1, LED_B1, LED_C1: footprint (none) -> ErgoDone:ERGO_LED-3MM
- R1, R2, RA1, RB1, RC1: footprint (none) -> ErgoDone:ERGO_RESISTOR
- S1, S2: footprint (none) -> ErgoDone:STAB_PCB940
- SW0:10, SW0:11, SW0:12, SW0:7, SW0:8, SW0:9, SW1:10, SW1:11, SW1:12, SW1:13, SW1:9, SW2:10, SW2:11, SW2:12, SW2:7, SW2:8, SW2:9, SW3:10, SW3:11, SW3:12, SW3:8, SW3:9, SW4:10, SW4:11, SW4:12, SW4:7, SW4:8, SW4:9, SW5:10, SW5:11, SW5:12, SW5:7, SW5:8, SW5:9: footprint (none) -> ErgoDone:MX_FLIP_DIODE_NOSMD; symbol SWITCH_DIODE-RESCUE-ErgoDOX -> SWITCH_DIODE
- SW2:13, SW3:13, SW4:13, SW5:13: footprint (none) -> ErgoDone:MX_FLIP_XX_NOSMD; symbol SWITCH_DIODE-RESCUE-ErgoDOX -> SWITCH_DIODE
- SX0:10, SX0:11, SX1:7, SX1:8: footprint (none) -> ErgoDone:MX_FLIP
- U1: footprint (none) -> ErgoDone:ProMicro
- U2: footprint (none) -> ErgoDone:MCP23017
Connections:
- net COL0: now also D71.2 (K), D72.2 (K), D73.2 (K), D74.2 (K), D75.2 (K), D76.2 (K), D77.2 (K), D78.2 (K), D79.2 (K), D80.2 (K)
- net COL1: now also D59.2 (K), D60.2 (K), D61.2 (K), D62.2 (K), D63.2 (K), D64.2 (K), D65.2 (K), D66.2 (K), D67.2 (K), D68.2 (K), D69.2 (K), D70.2 (K)
- net COL10: now also D35.2 (K), D36.2 (K), D37.2 (K), D38.2 (K), D39.2 (K), D40.2 (K), D41.2 (K), D42.2 (K), D43.2 (K), D44.2 (K), D45.2 (K), D46.2 (K)
- net COL11: now also D47.2 (K), D48.2 (K), D49.2 (K), D50.2 (K), D51.2 (K), D52.2 (K), D53.2 (K), D54.2 (K), D55.2 (K), D56.2 (K), D57.2 (K), D58.2 (K)
- net COL4: now also D23.2 (K), D24.2 (K), D25.2 (K), D26.2 (K), D27.2 (K), D28.2 (K), D29.2 (K), D30.2 (K), D31.2 (K), D32.2 (K), D33.2 (K), D34.2 (K)
- net COL5: now also D11.2 (K), D12.2 (K), D13.2 (K), D14.2 (K), D15.2 (K), D16.2 (K), D17.2 (K), D18.2 (K), D19.2 (K), D20.2 (K), D21.2 (K), D22.2 (K), D82.2 (K)
- net COL6: now also D1.2 (K), D10.2 (K), D2.2 (K), D3.2 (K), D4.2 (K), D5.2 (K), D6.2 (K), D7.2 (K), D8.2 (K), D81.2 (K), D9.2 (K)
- net GND: now also SW0:10.0 (GND), SW0:11.0 (GND), SW0:12.0 (GND), SW0:7.0 (GND), SW0:8.0 (GND), SW0:9.0 (GND), SW1:10.0 (GND), SW1:11.0 (GND), SW1:12.0 (GND), SW1:13.0 (GND), SW1:9.0 (GND), SW2:10.0 (GND), SW2:11.0 (GND), SW2:12.0 (GND), SW2:13.0 (GND), SW2:7.0 (GND), SW2:8.0 (GND), SW2:9.0 (GND), SW3:10.0 (GND), SW3:11.0 (GND), SW3:12.0 (GND), SW3:13.0 (GND), SW3:8.0 (GND), SW3:9.0 (GND), SW4:10.0 (GND), SW4:11.0 (GND), SW4:12.0 (GND), SW4:13.0 (GND), SW4:7.0 (GND), SW4:8.0 (GND), SW4:9.0 (GND), SW5:10.0 (GND), SW5:11.0 (GND), SW5:12.0 (GND), SW5:13.0 (GND), SW5:7.0 (GND), SW5:8.0 (GND), SW5:9.0 (GND)
- net at SW0:10.2, SW0:10.3 (A), SX0:10.2: now also D45.1 (A), D46.1 (A)
- net at SW4:7.2, SW4:7.3 (A): now also D3.1 (A), D4.1 (A)
- net at SW4:8.2, SW4:8.3 (A): now also D13.1 (A), D14.1 (A)
- net at SW4:12.2, SW4:12.3 (A): now also D61.1 (A), D62.1 (A)
- net at SW4:11.2, SW4:11.3 (A): now also D49.1 (A), D50.1 (A)
- net at SW4:10.2, SW4:10.3 (A): now also D37.1 (A), D38.1 (A)
- net at SW4:9.2, SW4:9.3 (A): now also D25.1 (A), D26.1 (A)
- net at SW4:13.2, SW4:13.3 (A): now also D73.1 (A), D74.1 (A)
- net at SW3:12.2, SW3:12.3 (A): now also D63.1 (A), D64.1 (A)
- net at SW3:11.2, SW3:11.3 (A): now also D51.1 (A), D52.1 (A)
- net at SW3:10.2, SW3:10.3 (A): now also D39.1 (A), D40.1 (A)
- net at SW3:9.2, SW3:9.3 (A): now also D27.1 (A), D28.1 (A)
- net at SW3:8.2, SW3:8.3 (A): now also D15.1 (A), D16.1 (A)
- net at SW1:9.2, SW1:9.3 (A): now also D31.1 (A), D32.1 (A)
- net at SW1:10.2, SW1:10.3 (A): now also D43.1 (A), D44.1 (A)
- net at SW1:12.2, SW1:12.3 (A): now also D67.1 (A), D68.1 (A)
- net at SW2:12.2, SW2:12.3 (A): now also D65.1 (A), D66.1 (A)
- net at SW2:11.2, SW2:11.3 (A): now also D53.1 (A), D54.1 (A)
- net at SW2:10.2, SW2:10.3 (A): now also D41.1 (A), D42.1 (A)
- net at SW2:9.2, SW2:9.3 (A): now also D29.1 (A), D30.1 (A)
- net at SW2:8.2, SW2:8.3 (A): now also D17.1 (A), D18.1 (A)
- net at SW2:7.2, SW2:7.3 (A): now also D5.1 (A), D6.1 (A)
- net at SW3:13.2, SW3:13.3 (A): now also D75.1 (A), D76.1 (A)
- net at SW1:13.2, SW1:13.3 (A): now also D79.1 (A), D80.1 (A)
- net at SW2:13.2, SW2:13.3 (A): now also D77.1 (A), D78.1 (A)
- net at SW0:11.2, SW0:11.3 (A), SX0:11.2: now also D57.1 (A), D58.1 (A)
- net at SW0:12.2, SW0:12.3 (A): now also D69.1 (A), D70.1 (A)
- net at SW0:7.2, SW0:7.3 (A): now also D10.1 (A), D9.1 (A)
- net at SW0:8.2, SW0:8.3 (A): now also D21.1 (A), D22.1 (A)
- net at SW0:9.2, SW0:9.3 (A): now also D33.1 (A), D34.1 (A)
- net at SW1:11.2, SW1:11.3 (A): now also D55.1 (A), D56.1 (A)
- net at SW5:13.2, SW5:13.3 (A): now also D71.1 (A), D72.1 (A)
- net at SW5:9.2, SW5:9.3 (A): now also D23.1 (A), D24.1 (A)
- net at SW5:10.2, SW5:10.3 (A): now also D35.1 (A), D36.1 (A)
- net at SW5:11.2, SW5:11.3 (A): now also D47.1 (A), D48.1 (A)
- net at SW5:12.2, SW5:12.3 (A): now also D59.1 (A), D60.1 (A)
- net at SW5:8.2, SW5:8.3 (A): now also D11.1 (A), D12.1 (A)
- net at SW5:7.2, SW5:7.3 (A): now also D1.1 (A), D2.1 (A)
- net at SX1:8.2: now also D19.1 (A), D20.1 (A), D82.1 (A)
- net at SX1:7.2: now also D7.1 (A), D8.1 (A), D81.1 (A)
